File: Mqtt.MordomusESP8266/HArdware/mordomusesp8266.brd (EAGLE design)
At the start: 83.9 x 99 mm, 41 parts, among them IC1 LM1117MPX-3.3, IC7 MCP23017SP, U2 MAX3232

Commit message: working pccwd API
Parts:
- moved R3 24.9 mm to (38.9, 49.3), turned to 0 degrees
- moved C4 13.6 mm to (1.27, 70.2), turned to 180 degrees
- moved C6 2.29 mm to (1.27, 73.0), turned to 180 degrees
- moved C2 1.42 mm to (1.27, 75.6), turned to 0 degrees
- moved C1 1.33 mm to (1.27, 78.1), turned to 0 degrees
- moved U2 1.27 mm to (7.62, 76.2)
- moved C7 1.08 mm to (13.2, 80.1), turned to 270 degrees
Connections:
- net +3V3: now also IC7.18
Routing:
- net +3V3: track 149.0 -> 169.7 mm
- net V+: track 5.85 -> 16.1 mm
- net GND: track 98.2 -> 92.1 mm
- net RX: track 28.3 -> 33.9 mm
- net TX: track 27.0 -> 32.2 mm
- net C1+: track 2.32 -> 6.71 mm
- net GPB0: track 18.8 -> 14.5 mm
- net C2+: track 2.29 -> 5.60 mm
- net RS232TX: track 33.9 -> 36.9 mm
- net RS232RX: track 37.9 -> 41.0 mm
- net SCL: track 49.6 -> 52.4 mm
- net GPB1: track 21.7 -> 19.2 mm
- net GPA2: track 46.5 -> 48.0 mm
- net GPA0: track 59.2 -> 60.7 mm
- net VDDR: track 151.8 -> 150.4 mm, vias 0 -> 1
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