File: Mqtt.MordomusESP8266/HArdware/mordomusesp8266.sch (EAGLE design)
At the start: 41 parts, among them IC1 LM1117MPX-3.3, IC7 MCP23017SP, U2 MAX3232

Commit message: working pccwd API
Connections:
- net +3V3: now also IC7.!RESET
Other:
- moved on the sheet: C4, C6, C7, X1
