File: Mqtt.ESP8266PlantConputer/HArdware - Copy/PlantComputerEsp8266.sch (EAGLE design)
At the start: 38 parts, among them IC1 LM1117MPX-3.3, Q1 BC337, Q2 BC337, U1 ULN2803AN

Commit message: stuff
Parts:
- R3: value (none) -> 15k
Connections:
- net SCL: now also SV1.3; no longer SV1.4
- net SDA: now also SV1.4; no longer SV1.3
Changed lines of the file:
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@@
 <part name="SV1" library="con-lstb" library_urn="urn:adsk.eagle:library:162" deviceset="MA10-1" device="" package3d_urn="urn:adsk.eagle:package:8346/1"/>
 <part name="U$1" library="Feesta-partsu" deviceset="OPTO-RELAY-CPC1017N" device=""/>
-<part name="R3" library="resistor" library_urn="urn:adsk.eagle:library:348" deviceset="R-EU_" device="R0805" package3d_urn="urn:adsk.eagle:package:23553/2"/>
+<part name="R3" library="resistor" library_urn="urn:adsk.eagle:library:348" deviceset="R-EU_" device="R0805" package3d_urn="urn:adsk.eagle:package:23553/2" value="15k"/>
 <part name="Q1" library="transistor-small-signal" library_urn="urn:adsk.eagle:library:401" deviceset="BC337" device="" package3d_urn="urn:adsk.eagle:package:29732/3"/>
 <part name="Q2" library="transistor-small-signal" library_urn="urn:adsk.eagle:library:401" deviceset="BC337" device="" package3d_urn="urn:adsk.eagle:package:29732/3"/>
@@
 </segment>
 <segment>
+<wire x1="50.8" y1="99.06" x2="43.18" y2="99.06" width="0.1524" layer="91"/>
+<label x="35.56" y="99.06" size="1.778" layer="95"/>
+<pinref part="SV1" gate="1" pin="3"/>
+</segment>
+</net>
+<net name="SDA" class="0">
+<segment>
+<pinref part="ESP" gate="G$1" pin="GPIO4"/>
+<wire x1="2.54" y1="-10.16" x2="10.16" y2="-10.16" width="0.1524" layer="91"/>
+<label x="10.16" y="-10.16" size="1.778" layer="95"/>
+</segment>
+<segment>
 <wire x1="50.8" y1="96.52" x2="43.18" y2="96.52" width="0.1524" layer="91"/>
 <label x="35.56" y="96.52" size="1.778" layer="95"/>
@@
 </segment>
 </net>
-<net name="SDA" class="0">
-<segment>
-<pinref part="ESP" gate="G$1" pin="GPIO4"/>
-<wire x1="2.54" y1="-10.16" x2="10.16" y2="-10.16" width="0.1524" layer="91"/>
-<label x="10.16" y="-10.16" size="1.778" layer="95"/>
-</segment>
-<segment>
-<wire x1="50.8" y1="99.06" x2="43.18" y2="99.06" width="0.1524" layer="91"/>
-<label x="35.56" y="99.06" size="1.778" layer="95"/>
-<pinref part="SV1" gate="1" pin="3"/>
-</segment>
-</net>
