File: HKMultiAccessory/Hardware/TRADFRIICC-1dimmer.brd (EAGLE design)
At the start: 39.4 x 66 mm, 14 parts

Commit message: Board updates
Parts:
- removed ESP: (no value), ESP8266-ESP12E:ESP8266-ESP12E
- removed PWR1: MP2307-MINI-360, MP2307-MINI-360:MP2307-MINI-360
- removed PWR_IN2: KF350-P2, KF350-P2:KF350-2P
- removed R1, R11, R12, R2: 10K, resistor:R0603
- removed S1: (no value), switch-omron:B3F-10XX
- removed SERIAL: (no value), con-lstb:MA04-1
- added IC1: LM1117MPX-3.3, lm1117:SOT223
- added JP1: (no value), pinhead:1_05X2MM
- added PWR_IN: KF350-P2, KF350-P2:KF350-2P
- C1: value (none) -> 100u; device resistor:E2-5 -> rcl:CT3528
- C2: value (none) -> 10u; device resistor:E2-5 -> rcl:C/6032-28R
- moved C1 70.9 mm to (12.1, 6.48), turned to 90 degrees
- moved R9 30.3 mm to (11.2, 18.4), turned to 180 degrees
- moved PWR_IN1 28.2 mm to (5.08, 29.2), turned to 180 degrees
- moved W 22.5 mm to (5.08, 16.5), turned to 180 degrees
- moved C2 21.6 mm to (5.08, 10.2)
Connections:
- removed net IRLED: ESP.20
- removed net N$2: ESP.10, R1.1
- removed net N$3: ESP.3, R11.2
- removed net PIR: ESP.19
- removed net PROG: ESP.12, R2.2, S1.3, S1.4
- removed net RX: ESP.15, SERIAL.2
- removed net TX: ESP.16, SERIAL.3
- removed net VCC: C1.+, C2.+, ESP.8, PWR1.3.3V, R11.1, R12.1, R2.1, SERIAL.1
- removed net W: ESP.7, R9.1
- new net +3V3: C1.+, IC1.2, IC1.TAB, JP1.5
- new net N$5: JP1.1
- new net PWM: JP1.3, R9.1
- net GND: now also IC1.1, JP1.4, PWR_IN.1; no longer ESP.9, PWR1.GND@1, PWR1.GND@2, PWR_IN2.2, R1.2, S1.1, S1.2, SERIAL.4
- net N$4: now also JP1.2; no longer ESP.11, R12.2
- net VDD: now also C2.+, IC1.3, PWR_IN.2; no longer PWR1.12V, PWR_IN2.1
Routing:
- net VDD: track 1.05 -> 46.4 mm
- net VCC: track 35.7 -> 0.00 mm, vias 4 -> 0
- net +3V3: track 0.00 -> 24.6 mm
- net GND: track 1.38 -> 21.9 mm, vias 0 -> 2
- net DW: track 1.15 -> 16.5 mm
- net RX: track 6.23 -> 0.00 mm
- net TX: track 5.97 -> 0.00 mm
- net PWM: track 0.00 -> 4.00 mm
- net PROG: track 3.03 -> 0.00 mm
- net N$4: track 2.88 -> 0.00 mm
- net N$13: track 0.00 -> 2.50 mm
- net N$2: track 2.48 -> 0.00 mm
- net W: track 1.33 -> 0.00 mm
- net N$3: track 1.13 -> 0.00 mm
- net PIR: track 0.74 -> 0.00 mm
Other:
- board size 39.4 x 66 mm -> 36.5 x 35.5 mm
- board text removed: "+"
- board text removed: "+ LED -"
- board text removed: "-"
- board text removed: "NB 2018 RGBWIRT v1.0"
- board text removed: "RX"
- board text removed: "TX"
- board text removed: "W"
