File: HKMultiAccessory/Hardware/TRADFRIICC-1dimmer.sch (EAGLE design)
At the start: 14 parts

Commit message: Board updates
Parts:
- removed ESP: (no value), ESP8266-ESP12E:ESP8266-12EESP8266-ESP12E
- removed PWR1: MP2307-MINI-360, MP2307-MINI-360:MP2307-MINI-360
- removed PWR_IN2: KF350-P2, KF350-P2:KF350-P2
- removed R1, R11, R12, R2: 10K, resistor:R-EU_R0603
- removed S1: (no value), switch-omron:10-XX
- removed SERIAL: (no value), con-lstb:MA04-1
- added IC1: LM1117MPX-3.3, lm1117:LM1117MPX-3.3
- added JP1: (no value), pinhead:PINHD-1X55X2MM
- added PWR_IN: KF350-P2, KF350-P2:KF350-P2
- C1: value (none) -> 100u; device resistor:CPOL-EUE2-5 -> rcl:CPOL-USCT3528
- C2: value (none) -> 10u; device resistor:CPOL-EUE2-5 -> rcl:CPOL-USC/6032-28R
Connections:
- removed net IRLED: ESP.GPIO10
- removed net N$2: ESP.GPIO15, R1.1
- removed net N$3: ESP.CH_PD, R11.2
- removed net PIR: ESP.GPIO9
- removed net PROG: ESP.GPIO0, R2.2, S1.P, S1.P1
- removed net RX: ESP.RXD, SERIAL.2
- removed net TX: ESP.TXD, SERIAL.3
- removed net VCC: C1.+, C2.+, ESP.VCC, PWR1.3.3V, R11.1, R12.1, R2.1, SERIAL.1
- removed net W: ESP.GPIO13, R9.1
- new net +3V3: C1.+, IC1.OUT, IC1.OUT1, JP1.5
- new net N$5: JP1.1
- new net PWM: JP1.3, R9.1
- net GND: now also IC1.GND, JP1.4, PWR_IN.1; no longer ESP.GND, PWR1.GND@1, PWR1.GND@2, PWR_IN2.2, R1.2, S1.S, S1.S1, SERIAL.4
- net N$4: now also JP1.2; no longer ESP.GPIO2, R12.2
- net VDD: now also C2.+, IC1.IN, PWR_IN.2; no longer PWR1.12V, PWR_IN2.1
Other:
- moved on the sheet: C1, C2
