File: PCCWDplus/circuit/mordomusesp8266.kicad_pcb (KiCad board)
At the start: 2 copper layers, 83.9 x 99 mm, 45 parts, among them IC1 LM1117MPX-3.3, IC7 MCP23017SP, U2 MAX3232

Commit message: Complete KiCad project + add WT0132C6-S5 symbol for ESP32-C6 revision
KiCad GUI 'Import Non-KiCad Project' created the full project from the
Eagle .sch: project file, schematic, merged symbol library, and refreshed
board. All 45 footprints, 278 tracks, 9 vias, and 6 zones imported cleanly
(ground pours just need 'B' to refill, which is normal).

Added hand-written symbol for the revision part:

  PCCWDplus/circuit/lib/WT0132C6-S5.kicad_sym

Wireless-Tag WT0132C6-S5 is an ESP32-C6 module in ESP-12F footprint,
pin-to-pin drop-in for the current ESP8266/ESP-12F module. Pin types and
numbering transcribed from the V1.0.1 datasheet; uses KiCad stdlib
footprint RF_Module:ESP-12F. Strapping pins (IO4/MTMS, IO5/MTDI, IO8, IO9)
are labeled with their alternate functions in the pin name.

Registered a project-local 'pccwd-local' library in sym-lib-table for
this symbol and any future hand-written parts.

.gitignore additions:
- KiCad auto-backups (*-backups/)
- fp-info-cache
- *.kicad_prl (per-user UI state)
- .history/ (VSCode Local History extension)

Co-Authored-By: Claude Opus 4.6 <noreply@anthropic.com>
Parts:
- moved C1 179.5 mm to (112.9, 62.5)
- moved C2 179.5 mm to (112.9, 65.0)
- moved C4 179.5 mm to (112.9, 70.3)
- moved C6 179.5 mm to (112.9, 67.5)
- moved C7 179.5 mm to (124.8, 60.4)
- moved D2 179.5 mm to (134.5, 135.5)
- moved ESP0 179.5 mm to (116.7, 96.1)
- moved IC1 179.5 mm to (138.3, 115.2)
- moved PWR1 179.5 mm to (143.5, 129.1)
- moved PWR_IN0 179.5 mm to (111.6, 139.3)
- moved PWR_IN14 179.5 mm to (111.6, 131.7)
- moved PWR_INBAT0 179.5 mm to (111.6, 146.9)
- moved R11 179.5 mm to (114.8, 107.5)
- moved R12 179.5 mm to (120.9, 83.3)
- moved R2 179.5 mm to (131.9, 107.5)
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Other:
- board size 83.9 x 99 mm -> 83.9 x 99.1 mm
- board text removed: "+"
- board text removed: "+12V"
- board text removed: "-"
- board text removed: "BAT"
- board text removed: "GND"
- board text removed: "GPA0"
- board text removed: "GPA1"
- board text removed: "GPA2"
- board text removed: "GPA3"
- board text removed: "GPA4"
- board text removed: "GPA5"
- board text removed: "GPA6"
- board text removed: "GPA7"
- board text removed: "GPB0"
- board text removed: "GPB1"
- board text removed: "GPB2"
- board text removed: "GPB3"
- board text removed: "GPB4"
- board text removed: "GPB5"
- board text removed: "GPB6"
- board text removed: "GPB7"
- board text removed: "LED"
- board text removed: "NB 2019 PCCW MQTT + IO + LED v1.1"
- board text removed: "POW"
- board text removed: "RX"
- board text removed: "SERIAL"
- board text removed: "TX"

Commit message: PCCWDplus: finish KiCad migration — net normalization, reset button, silk recovery
- Swap ESP8266-12E symbol for WT0132C6-S5 (ESP32-C6) drop-in; pin tips
  match ESP-12F exactly so existing wiring is preserved
- Normalize power net: collapse VCC / 3.3V / +3V3 mess to a single +3V3
  across schematic, PCB, and zones; fix dangling R3/R4 I²C pull-up pads
- Add S2 reset button; switch both S1/S2 to stock Switch:SW_Push symbol
  and Button_Switch_THT:SW_PUSH_6mm_H7.3mm footprint (Omron B3F-10XX eq.)
- Recover silkscreen lost on Eagle import: merge fp_line/arc/circle/poly/
  rect/text from a fresh re-import, plus shifted board-level gr_text
  (pin labels on screw terminals, +12V/GND/GPA*/GPB*, TX/RX, title block)
- Un-hide component reference designators to match original silk

Co-Authored-By: Claude Opus 4.7 <noreply@anthropic.com>
Parts:
- removed R1, R12: 10K, R0603
- removed UNK_HOLE_0: , dummyfp0
- removed UNK_HOLE_1: , dummyfp1
- removed UNK_HOLE_2: , dummyfp2
- removed UNK_HOLE_3: , dummyfp3
- C3, C5: value (none) -> 100UF-25V-20%(PTH)
- D1, D2: value (none) -> SCHOTTKY-DIODESMC
- ESP0: value (none) -> WT0132C6-S5
- G0: value (none) -> FDS5680
- IC1: value LM1117MPX-3.3 -> LM1117MPX-
- S1: value (none) -> 10-XX
- SERIAL0: value (none) -> MA04-1
- X1: value (none) -> M09HP
Connections:
- net C1+ renamed Net-(U2-C1+)
- net C1- renamed Net-(U2-C1-)
- net C2+ renamed Net-(U2-C2+)
- net C2- renamed Net-(U2-C2-)
- net DG renamed Net-(G0-D-Pad5)
- net GPA0 renamed /GPA0
- net GPA1 renamed /GPA1
- net GPA2 renamed /GPA2
- net GPA3 renamed /GPA3
- net GPA4 renamed /GPA4
- net GPA5 renamed /GPA5
- net GPA6 renamed /GPA6
- net GPA7 renamed /GPA7
- net GPB0 renamed /GPB0
- net GPB1 renamed /GPB1
- net GPB2 renamed /GPB2
- net GPB3 renamed /GPB3
- net GPB4 renamed /GPB4
- net GPB5 renamed /GPB5
- net GPB6 renamed /GPB6
- net GPB7 renamed /GPB7
- net INTA renamed /INTA
- net INTB renamed /INTB
- net PROG renamed /PROG
- net RS232RX renamed /RS232RX
- net RS232TX renamed /RS232TX
- net RVCC renamed Net-(C3-+)
- net SCL renamed /SCL
- net SDA renamed /SDA
- net V+ renamed Net-(U2-V+)
- net V- renamed Net-(U2-V-)
- net VDD renamed /VDD
- net VDDBAT renamed /VDDBAT
- net VDDR renamed /VDDR
- net W renamed /W
- ESP0 pad 1: (no net) -> /TX_2
- ESP0 pad 10: N$2 -> unconnected-(ESP0-IO19-Pad10)
- ESP0 pad 11: N$4 -> unconnected-(ESP0-IO20-Pad11)
- ESP0 pad 15: RX -> /RX
- ESP0 pad 16: TX -> /TX
- ESP0 pad 17: (no net) -> unconnected-(ESP0-IO8-Pad17)
- ESP0 pad 18: (no net) -> unconnected-(ESP0-IO9-Pad18)
- ESP0 pad 19: (no net) -> unconnected-(ESP0-IO10-Pad19)
- ESP0 pad 2: (no net) -> /RX_2
- ESP0 pad 20: (no net) -> unconnected-(ESP0-IO3-Pad20)
- ESP0 pad 21: (no net) -> unconnected-(ESP0-U0RXD/IO17-Pad21)
- ESP0 pad 22: (no net) -> unconnected-(ESP0-U0TXD/IO16-Pad22)
- ESP0 pad 5: (no net) -> unconnected-(ESP0-IO4/MTMS-Pad5)
- SERIAL0 pad 2: RX -> /RX_2
- SERIAL0 pad 3: TX -> /TX_2
- U2 pad 10: (no net) -> unconnected-(U2-T2IN-Pad10)
- U2 pad 11: TX -> /TX
- U2 pad 12: RX -> /RX
- U2 pad 7: (no net) -> unconnected-(U2-T2OUT-Pad7)
- U2 pad 8: (no net) -> unconnected-(U2-R2IN-Pad8)
- U2 pad 9: (no net) -> unconnected-(U2-R2OUT-Pad9)
- X1 pad 1: (no net) -> unconnected-(X1-Pad1)
- X1 pad 4: (no net) -> unconnected-(X1-Pad4)
- X1 pad 6: (no net) -> unconnected-(X1-Pad6)
- X1 pad 7: (no net) -> unconnected-(X1-Pad7)
- X1 pad 8: (no net) -> unconnected-(X1-Pad8)
- X1 pad 9: (no net) -> unconnected-(X1-Pad9)
Routing:
- net RX: track 33.9 -> 0.00 mm
- net TX: track 32.2 -> 0.00 mm
- net /RX_2: track 0.00 -> 30.7 mm
- net /TX_2: track 0.00 -> 30.5 mm
- net /RX: track 0.00 -> 30.0 mm
- net /TX: track 0.00 -> 29.6 mm
- net GND: track 92.1 -> 86.8 mm
- net N$2: track 4.49 -> 0.00 mm
- net +3V3: track 169.7 -> 166.0 mm
- net N$4: track 3.41 -> 0.00 mm
Other:
- board text added: "+"
- board text added: "+12V"
- board text added: "-"
- board text added: "BAT"
- board text added: "GND"
- board text added: "GPA0"
- board text added: "GPA1"
- board text added: "GPA2"
- board text added: "GPA3"
- board text added: "GPA4"
- board text added: "GPA5"
- board text added: "GPA6"
- board text added: "GPA7"
- board text added: "GPB0"
- board text added: "GPB1"
- board text added: "GPB2"
- board text added: "GPB3"
- board text added: "GPB4"
- board text added: "GPB5"
- board text added: "GPB6"
- board text added: "GPB7"
- board text added: "LED"
- board text added: "NB 2019 PCCW MQTT + IO + LED v1.1"
- board text added: "POW"
- board text added: "RX"
- board text added: "SERIAL"
- board text added: "TX"
