File: PCCWDplus/circuit/mordomusesp8266.kicad_sch (KiCad schematic)
At the start: 41 parts, among them IC1 LM1117MPX-, IC7 MCP23017SP, U2 MAX3232, X1 M09HP

Commit message: PCCWDplus: finish KiCad migration — net normalization, reset button, silk recovery
- Swap ESP8266-12E symbol for WT0132C6-S5 (ESP32-C6) drop-in; pin tips
  match ESP-12F exactly so existing wiring is preserved
- Normalize power net: collapse VCC / 3.3V / +3V3 mess to a single +3V3
  across schematic, PCB, and zones; fix dangling R3/R4 I²C pull-up pads
- Add S2 reset button; switch both S1/S2 to stock Switch:SW_Push symbol
  and Button_Switch_THT:SW_PUSH_6mm_H7.3mm footprint (Omron B3F-10XX eq.)
- Recover silkscreen lost on Eagle import: merge fp_line/arc/circle/poly/
  rect/text from a fresh re-import, plus shifted board-level gr_text
  (pin labels on screw terminals, +12V/GND/GPA*/GPB*, TX/RX, title block)
- Un-hide component reference designators to match original silk

Co-Authored-By: Claude Opus 4.7 <noreply@anthropic.com>
Parts:
- removed R1, R12: 10K, mordomusesp8266:R0603, symbol mordomusesp8266-eagle-import:R-EU_R0603
- removed S1: 10-XX, mordomusesp8266:B3F-10XX, symbol mordomusesp8266-eagle-import:10-XX
- added SW1, SW2: SW_Push, Button_Switch_THT:SW_TH_Tactile_Omron_B3F-100x, symbol Switch:SW_Push
- ESP0: value ESP8266-12EESP8266-ESP12E -> WT0132C6-S5; footprint mordomusesp8266:ESP8266-ESP12E -> RF_Module:ESP-12F; symbol mordomusesp8266-eagle-import:ESP8266-12EESP8266-ESP12E -> pccwd-local:WT0132C6-S5
Connections:
- net VCC is gone; now on net +3V3: C5.1 (+), C7.1, IC1.2 (OUT), IC1.TAB (OUT1), U2.16 (VCC)
- net GND: now also SW1.2, SW2.2
- net PROG: now also SW1.1
- net RX: no longer SERIAL0.2
- net TX: no longer SERIAL0.3
- net TX_2: now reaches ESP0.1 (IO0)
- net TX_2: now also SERIAL0.3
- net RX_2: now reaches ESP0.2 (IO1)
- net RX_2: now also SERIAL0.2
- net EN: now reaches ESP0.3 (EN), R11.2
- net EN: now also SW2.1
- net 3.3V renamed +3V3
Other:
- moved on the sheet: R11, R2
