File: ESP32C6_ZIGBEE_Wall_Input_Module/circuit/ESP32C6_Wall_Input_Module.kicad_pcb (KiCad board)
At the start: 2 copper layers, 45 x 36 mm, 26 parts, among them J1 MAINS IN, J2 WALL SWITCHES, J3 PROG, SW3 BOOT, U1 HLK-PM01, U2 AMS1117-3.3, U3 WT0132C6-S5

Commit message: C6: 100µF→47µF to fit the Ø4 footprint (sourceable part)
100µF SMD electrolytics only come in Ø6.3mm cans, which don't fit C6's
Ø4 footprint. Drop C6 to 47µF/16V (LCSC C3337, Ø5 can solders to the Ø4
pads by hand) — it's supplementary 3V3 bulk near the module, non-critical.
Value-only change; bare board already ordered, footprint unchanged.

Co-Authored-By: Claude Opus 4.8 <noreply@anthropic.com>
Parts:
- C6: value 100u -> 47u
Changed lines of the file:
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@@
 			)
 		)
-		(property "Value" "100u"
+		(property "Value" "47u"
 			(at 0 -3.2 270)
 			(layer "B.Fab")

Commit message: Wall Input Module: scene-switch actions + Zigbee OTA + corrected WT pinout
Firmware: convert the two inputs from IAS contact sensors to a Hue/Modomus-
style scene switch — per-input single/double/long gesture detection reported
via Multistate Input (genMultistateInput presentValue 1/2/3). Add a Zigbee OTA
client on EP10; requestOTAUpdate() is started from loop() after the mesh is up.

Converter: expose button actions (button_1/2_single|double|hold) instead of
contact; bind genMultistateInput in configure() so reports reach Z2M; drop
duplicate reports with a 250ms time-dedup; declare ota:true.

Schematic/PCB: correct the WT0132C6-S5 symbol pin numbering (TXD/RXD/IO9 etc.
were on the wrong pins) and reroute the board to match. Footprint pad map was
already correct and is unchanged.

Verified end-to-end on hardware: joins Z2M, reports single/double/long per
button, and OTA-updated itself from v1.0.0.0 to v1.0.0.1 over the air.

Co-Authored-By: Claude Opus 4.8 <noreply@anthropic.com>
Parts:
- C1: footprint CP_Elec_6.3x5.4 -> Capacitor_SMD:CP_Elec_6.3x5.4
- C10, C2, C3, C5, C7, C8, C9: footprint C_0805_2012Metric -> Capacitor_SMD:C_0805_2012Metric
- C4: footprint CP_EIA-3528-21_Kemet-B -> Capacitor_Tantalum_SMD:CP_EIA-3528-21_Kemet-B
- C6: footprint CP_Elec_4x5.4 -> Capacitor_SMD:CP_Elec_4x5.4
- F1: footprint Fuse_Littelfuse_395Series -> Fuse:Fuse_Littelfuse_395Series
- J1: footprint TerminalBlock_Phoenix_MKDS-3-2-5.08_1x02_P5.08mm_Horizontal -> TerminalBlock_Phoenix:TerminalBlock_Phoenix_MKDS-3-2-5.08_1x02_P5.08mm_Horizontal
- J2: footprint TerminalBlock_Phoenix_MKDS-1,5-3-5.08_1x03_P5.08mm_Horizontal -> TerminalBlock_Phoenix:TerminalBlock_Phoenix_MKDS-1,5-3-5.08_1x03_P5.08mm_Horizontal
- J3: footprint PinHeader_1x06_P1.27mm_Vertical -> Connector_PinHeader_1.27mm:PinHeader_1x06_P1.27mm_Vertical
- LED1: footprint LED_0805_2012Metric -> LED_SMD:LED_0805_2012Metric
- R1, R2, R3, R4, R5, R6: footprint R_0805_2012Metric -> Resistor_SMD:R_0805_2012Metric
- RV1: footprint RV_Disc_D7mm_W3.5mm_P5mm -> Varistor:RV_Disc_D7mm_W3.5mm_P5mm
- SW3: footprint SW_SPST_TL3342 -> Button_Switch_SMD:SW_SPST_TL3342
- U1: footprint Converter_ACDC_Hi-Link_HLK-PMxx -> Converter_ACDC:Converter_ACDC_Hi-Link_HLK-PMxx
- U2: footprint SOT-223-3_TabPin2 -> Package_TO_SOT_SMD:SOT-223-3_TabPin2
- U3: footprint WT0132C6-S5 -> WT0132:WT0132C6-S5
Connections:
- U3 pad 10: unconnected-(U3-IO19-Pad10) -> /STATUS_LED
- U3 pad 12: unconnected-(U3-IO21-Pad12) -> /IO9
- U3 pad 15: /STATUS_LED -> /RXD0
- U3 pad 16: unconnected-(U3-IO7/MTDO-Pad16) -> /TXD0
- U3 pad 18: /IO9 -> unconnected-(U3-IO19-Pad18)
- U3 pad 21: /RXD0 -> unconnected-(U3-IO22-Pad21)
- U3 pad 22: /TXD0 -> unconnected-(U3-IO23-Pad22)
Routing:
- net /STATUS_LED: track 28.5 -> 18.0 mm
- net /IO9: track 44.3 -> 52.5 mm, vias 1 -> 2
- net /RXD0: track 28.9 -> 22.9 mm
- net /TXD0: track 24.1 -> 29.6 mm
