File: ESP32C6_ZIGBEE_Wall_Input_Module/circuit/ESP32C6_Wall_Input_Module.kicad_sch (KiCad schematic)
At the start: 26 parts, among them J1 MAINS IN, J2 WALL SWITCHES, J3 PROG, SW3 BOOT, U1 HLK-PM01, U2 AMS1117-3.3, U3 WT0132C6-S5

Commit message: C6: 100µF→47µF to fit the Ø4 footprint (sourceable part)
100µF SMD electrolytics only come in Ø6.3mm cans, which don't fit C6's
Ø4 footprint. Drop C6 to 47µF/16V (LCSC C3337, Ø5 can solders to the Ø4
pads by hand) — it's supplementary 3V3 bulk near the module, non-critical.
Value-only change; bare board already ordered, footprint unchanged.

Co-Authored-By: Claude Opus 4.8 <noreply@anthropic.com>
Parts:
- C6: value 100u -> 47u
Changed lines of the file:
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@@
 			)
 		)
-		(property "Value" "100u"
+		(property "Value" "47u"
 			(at 159.766 105.41 0)
 			(effects

Commit message: Wall Input Module: scene-switch actions + Zigbee OTA + corrected WT pinout
Firmware: convert the two inputs from IAS contact sensors to a Hue/Modomus-
style scene switch — per-input single/double/long gesture detection reported
via Multistate Input (genMultistateInput presentValue 1/2/3). Add a Zigbee OTA
client on EP10; requestOTAUpdate() is started from loop() after the mesh is up.

Converter: expose button actions (button_1/2_single|double|hold) instead of
contact; bind genMultistateInput in configure() so reports reach Z2M; drop
duplicate reports with a 250ms time-dedup; declare ota:true.

Schematic/PCB: correct the WT0132C6-S5 symbol pin numbering (TXD/RXD/IO9 etc.
were on the wrong pins) and reroute the board to match. Footprint pad map was
already correct and is unchanged.

Verified end-to-end on hardware: joins Z2M, reports single/double/long per
button, and OTA-updated itself from v1.0.0.0 to v1.0.0.1 over the air.

Co-Authored-By: Claude Opus 4.8 <noreply@anthropic.com>
Connections:
- net IO9: now also U3.12 (IO9); no longer U3.18 (IO9)
- net RXD0: now also U3.15 (RXD); no longer U3.21 (U0RXD/IO17)
- net STATUS_LED: now also U3.10 (IO7); no longer U3.15 (IO18)
- net TXD0: now also U3.16 (TXD); no longer U3.22 (U0TXD/IO16)
- no-connect marks 13 -> 16
